File: hardware/EBike_Smart_Controller.sch (KiCad schematic (older format))
At the start: 39 parts, among them IC1 ACS756SCA-100B, K1 Throttle, P1 Brake, P2 Hall sensors, P3 Zero LPC2103 board, P4 BLUETOOTH_MODULE, P5 CONN_10, P6 CONN_10

Commit message: Started to working on Prototype V2. Added 12V DC-DC to schematic.
Parts:
- removed P6: CONN_10, symbol CONN_10
- added C10, C11: 100nF, symbol C_MINI
- added C12, C9: 47uF, symbol CAPAPOL
- added D1, D2: PMEG6010, symbol D_SCHOTTKY
- added L1: 100uH, symbol L_MINI
- added P6: Battery input, symbol CONN_2
- added P7: CONN_11, symbol CONN_11
- added R24: 92k 1%, symbol R_MINI
- added R25: 10k 1%, symbol R_MINI
- added U1: MAX5035, symbol MAX5035
Connections:
- net labels added: +12V, Battery +, Mosfets_temperature_signal (LPC2103 P0.??)
- wire segments 124 -> 177
Other:
- note added: "MAX5035D"
- note removed: "(C28)"
- note removed: "(CPU32)"
- note removed: "(CPU33)"
- note removed: "(R50)"
- note removed: "(R55)"
- note removed: "(R56)"
- note removed: "KU63 controller"
- note removed: "Note: 5V power source is from KU63 controller."
- note removed: "Note: exchange R46 (shunt resistor) by this current sensor IC."
- note removed: "Note: please refer to KU63 schematic."
- moved on the sheet: C1, C2, C3, C4, C5, C6, C7, C8, IC1, K1, P1, P2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
