File: hardware/EBike_Smart_Controller.sch (KiCad schematic (older format))
At the start: 50 parts, among them IC1 ACS756SCA-100B, K1 Throttle, P1 Brake, P2 Hall sensors, P3 Zero LPC2103 board, P4 BLUETOOTH_MODULE, P5 CONN_10, P6 Battery input, P7 CONN_11, U1 MAX5035

Commit message: More work on schematic.
Parts:
- added C13, C14, C15, C16, C18, C19, C20: 100nF, symbol C_MINI
- added C17: 10nF, symbol C_MINI
- added C21: 1uF, symbol CAPAPOL
- added D3, D4, D5: PMEG6010, symbol D_SCHOTTKY
- added Q1, Q2, Q3, Q4, Q5, Q6: MOSFET_N_OPENDOUS, symbol MOSFET_N_OPENDOUS
- added R26: 3K6 1%, symbol R_MINI
- added R27: 6K8 1%, symbol R_MINI
- added R28, R29, R30, R31, R32, R33: 10R, symbol R_MINI
- added R34, R38, R39: 100k, symbol R_MINI
- added R35: 100K, symbol R_MINI
- added R36, R37: 10k, symbol R_MINI
- added U2: LM50, symbol LM50
- added U3, U4, U5: IR2181, symbol IR2181
- added U6: 78L05, symbol 78L05
Connections:
- net labels added: IO for mosfet phase_c high (LPC2103 P0.19), Motor Phase A, Motor Phase B, Motor Phase C
- net labels removed: Battery +
- wire segments 177 -> 310
Other:
- note added: "EBike Smart Controller main control board"
- note removed: "(CPU1)"
- note removed: "(CPU2)"
- note removed: "(CPU3)"
- note removed: "(CPU4)"
- note removed: "(CPU44)"
- note removed: "(CPU5)"
- note removed: "EBike Smart Controller main board"
- moved on the sheet: C10, C11, C2, C4, C5, IC1, P6, R11, R12, R24, R25, R4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

Commit message: Final schematic of prototype V2 (untested).
Parts:
- removed P5: CONN_10, symbol CONN_10
- added P5: CONN_11, symbol CONN_11
- Q1, Q2, Q3, Q4, Q5, Q6: value MOSFET_N_OPENDOUS -> PSMN6R5-80PS
- R18, R19, R20: value 10K -> 100k
- R21, R22, R23, R36, R37: value 10k -> 100k
Connections:
- net labels added: Mosfets_temperature_signal (LPC2103 P0.25)
- net labels removed: Mosfets_temperature_signal (LPC2103 P0.??)
- wire segments 310 -> 263
Other:
- note added: "EBike Smart Controller control board"
- note added: "EBike Smart Controller power board"
- note removed: "EBike Smart Controller main control board"
- moved on the sheet: C1, C10, C11, C13, C14, C15, C16, C17, C18, C19, C2, C20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

Commit message: Updated schematic.
Parts:
- removed Q3, Q4, Q5, Q6: PSMN6R5-80PS, symbol MOSFET_N_OPENDOUS
- removed R35: 100K, symbol R_MINI
- removed R36, R38, R39: 100k, symbol R_MINI
- added C? (x2): 3300uF, symbol CAPAPOL
- added Q? (x4): PSMN6R5-80PS, symbol MOSFET_N_OPENDOUS
- added R? (x2): 100k, symbol R_MINI
- added R? (x2): 100K, symbol R_MINI
- R34: value 100k -> 100K
Connections:
- wire segments 263 -> 333
Other:
- moved on the sheet: C14, C15, C16, C18, C19, C20, R18, R19, R20, R21, R22, R23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
