File: hardware/EBike_Smart_Controller.sch (KiCad schematic (older format))
At the start: 89 parts, among them IC1 ACS756SCA-100B, K1 Throttle, P1 Brake, P2 Hall sensors, P3 Zero LPC2103 board, P4 BLUETOOTH_MODULE, P5 CONN_11, P6 Battery input, P7 CONN_11, Q1 PSMN6R5-80PS, Q2 PSMN6R5-80PS, U1 MAX5035, U2 LM50, U3 IR2181, U4 IR2181, U5 IR2181, U6 78L05

Commit message: Changes to schematic to update with current prototype 2.
Parts:
- removed P5, P7: CONN_11, symbol CONN_11
- removed Q1, Q2, Q? (x4): PSMN6R5-80PS, symbol MOSFET_N_OPENDOUS
- added C18: 100nF, symbol C_MINI
- added Q1, Q2, Q3, Q4, Q5, Q6: PSMN6R5-80PS, symbol PSMN6R5-80PS
- gave numbers to parts that had none: 6
- renumbered C4 to C1, C16 to C10, C13 to C11, C11 to C12, C18 to C13, C19 to C14, C20 to C15, C17 to C16, C12 to C17, C21 to C19, C1 to C20, C3 to C21, C6 to C22, C7 to C23, C8 to C24, C9 to C6, C10 to C7, C14 to C8, C15 to C9, D3 to D2, D4 to D3, D5 to D4, D2 to D5, P6 to P1, P2 to P3, P1 to P4, P3 to P6, P4 to P7, R6 to R1, R21 to R10, R22 to R11, R23 to R12, R26 to R13, R27 to R14, R28 to R15, R29 to R16, R30 to R17, R31 to R18, R32 to R19, R7 to R2, R33 to R20, R24 to R21, R25 to R22, R37 to R23, R34 to R24, R1 to R29, R11 to R3, R8 to R30, R2 to R31, R3 to R32, R13 to R33, R9 to R34, R10 to R35, R14 to R36, R15 to R37, R16 to R38, R17 to R39, R12 to R6, R18 to R7, R19 to R8, R20 to R9, U3 to U2, U4 to U3, U5 to U4, U2 to U5
Connections:
- net labels added: Battery GND
- wire segments 333 -> 318
Other:
- note added: "This is the circuit GND."
- note removed: "Battery GND"
- note removed: "EBike Smart Controller control board"
- note removed: "EBike Smart Controller power board"
- moved on the sheet: C1, C10, C11, C12, C13, C14, C15, C16, C2, C20, C21, C22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

Commit message: Updates to schematic.
Connections:
- net labels removed: Motor GND
- wire segments 318 -> 312

Commit message: Changes on schematic to add the BIG 10mF capacitor. This is now for prototype 3
Parts:
- removed C4: 3300uF, symbol CAPAPOL
- added C? (x4): 10uF, symbol C_MINI
- C3: value 3300uF -> 10mF
Connections:
- wire segments 312 -> 322
Other:
- moved on the sheet: C12, C18, C22, C23, C24, C7, P1, P3, R21, R22, R30, R34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

Commit message: Modified schematic for prototype V3 (using the STM32F100 instead LPC2103).
Parts:
- removed P6: Zero LPC2103 board, symbol CONN_20X2
- added P2: EXT1, symbol CONN_8X2
- added P5: EXT2, symbol CONN_8X2
- IC1: value ACS756SCA-100B -> ACS756SCA-050B
- R30, R35: value 2K2 -> 3K6
- R34: value 2K2 -> 6K8 1%
- R37, R39: value 3K6 -> 6K8 1%
- gave numbers to parts that had none: 4
Connections:
- net labels added: Brake_signal (STM32F100 PB12), Current_signal (STM32F100 PA2), Hall sensor phase_a (STM32F100 PA6), Hall sensor phase_b (STM32F100 PA7), Hall sensor phase_c (STM32F100 PB0), Mosfets_temperature_signal (STM32F100 PA3), PWM for mosfet phase_a high (STM32F100 PA8), PWM for mosfet phase_a low (STM32F100 PB13), PWM for mosfet phase_b high (STM32F100 PA9), PWM for mosfet phase_b low (STM32F100 PB14), PWM for mosfet phase_c high (STM32F100 PA10), PWM for mosfet phase_c low (STM32F100 PB15), Throttle_signal (STM32F100 PA0), UART RX (STM32F100 PB11), UART TX (STM32F100 PB10), Voltage_signal (STM32F100 PA1)
- net labels removed: Brake_signal (LPC2103 P0.11), Current_signal (LPC2103 P0.23), Hall sensor phase_a (LPC2103 P0.2), Hall sensor phase_b (LPC2103 P0.4), Hall sensor phase_c (LPC2103 P0.6), IO for mosfet phase_a high (LPC2103 P0.7), IO for mosfet phase_b high (LPC2103 P0.8), IO for mosfet phase_c high (LPC2103 P0.19), IO for mosfet phase_c high (LPC2103 P0.9), Mosfets_temperature_signal (LPC2103 P0.25), PWM for mosfet phase_a low (LPC2103 P0.12), PWM for mosfet phase_b low (LPC2103 P0.13), PWM for mosfet phase_c low (LPC2103 P0.19), Throttle_signal (LPC2103 P0.24), UART RX (LPC2103 P0.1), UART TX (LPC2103 P0.0), Voltage_signal (LPC2103 P0.22)
- wire segments 322 -> 323
- no-connect marks 55 -> 43
Other:
- note added: "Note: 3V3 power\nsource is from\nSTM32F100\nheader board."
- note added: "STM32F100\n(Bravekit.com Header board)"
- note removed: "Note: 3V3 power\nsource is from\nZero LPC2103\nboard."
- note removed: "Note: LPC2103 pins are 5V tolerant."
- note removed: "Zero LPC2103 board"
- note removed: "solder to LPC2103 board Vcc input"
- moved on the sheet: P3
